File: elec/layout/default/the-everything-sensor.kicad_pcb (KiCad board)
At the start: 2 copper layers, 225.7 x 100.8 mm, 0 parts

Commit message: layout complete
Parts:
- added C1: Multilayer Ceramic Capacitors MLCC - SMD/SMT 100nF 10V 0402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, lib:C0402, F.Cu at (147.9, 84.0)
- added C10: Multilayer Ceramic Capacitors MLCC - SMD/SMT 1uF 6.3V 0402 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, lib:C0402, F.Cu at (137.6, 104.9)
- added C11: Multilayer Ceramic Capacitors MLCC - SMD/SMT 100nF 10V 0402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, lib:C0402, F.Cu at (117.3, 54.9)
- added C12: Multilayer Ceramic Capacitors MLCC - SMD/SMT 10uF 10V 0805 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, lib:C0805, F.Cu at (115.8, 54.8)
- added C13: Multilayer Ceramic Capacitors MLCC - SMD/SMT 10uF 10V 0805 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, lib:C0805, F.Cu at (113.7, 54.8)
- added C14: Multilayer Ceramic Capacitors MLCC - SMD/SMT 20pF 50V 0402 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, lib:C0402, F.Cu at (179.8, 68.4)
- added C15: Multilayer Ceramic Capacitors MLCC - SMD/SMT 20pF 50V 0402 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, lib:C0402, F.Cu at (180.6, 63.1)
- added C16: Multilayer Ceramic Capacitors MLCC - SMD/SMT 100nF 10V 0402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, lib:C0402, F.Cu at (178.7, 63.0)
- added C17: Multilayer Ceramic Capacitors MLCC - SMD/SMT 100nF 10V 0402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, lib:C0402, F.Cu at (168.9, 59.0)
- added C18: Multilayer Ceramic Capacitors MLCC - SMD/SMT 100nF 10V 0402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, lib:C0402, F.Cu at (167.8, 69.6)
- added C19: Multilayer Ceramic Capacitors MLCC - SMD/SMT 100nF 10V 0402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, lib:C0402, F.Cu at (168.9, 69.6)
- added C2: Multilayer Ceramic Capacitors MLCC - SMD/SMT 2.2uF 10V 0603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, lib:C0603, F.Cu at (148.0, 85.3)
- added C20: Multilayer Ceramic Capacitors MLCC - SMD/SMT 100nF 10V 0402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, lib:C0402, F.Cu at (172.7, 58.9)
- added C21: Multilayer Ceramic Capacitors MLCC - SMD/SMT 1uF 6.3V 0402 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, lib:C0402, F.Cu at (159.6, 60.6)
- added C22: Multilayer Ceramic Capacitors MLCC - SMD/SMT 100nF 10V 0402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, lib:C0402, F.Cu at (166.4, 64.3)
- added C23: Multilayer Ceramic Capacitors MLCC - SMD/SMT 100nF 10V 0402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, lib:C0402, F.Cu at (167.8, 59.0)
- added C24: Multilayer Ceramic Capacitors MLCC - SMD/SMT 100nF 10V 0402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, lib:C0402, F.Cu at (178.7, 62.0)
- added C25: Multilayer Ceramic Capacitors MLCC - SMD/SMT 1uF 6.3V 0402 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, lib:C0402, F.Cu at (178.7, 60.9)
- added C26: Multilayer Ceramic Capacitors MLCC - SMD/SMT 1uF 6.3V 0402 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, lib:C0402, F.Cu at (164.5, 52.2)
- added C27: Multilayer Ceramic Capacitors MLCC - SMD/SMT 1uF 6.3V 0402 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, lib:C0402, F.Cu at (160.0, 52.1)
- added C28: Multilayer Ceramic Capacitors MLCC - SMD/SMT 2.2uF 100V 121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, lib:C1210, F.Cu at (142.5, 130.0)
- added C29: Multilayer Ceramic Capacitors MLCC - SMD/SMT 2.2uF 100V 121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, lib:C1210, F.Cu at (134.7, 130.0)
- added C3: Multilayer Ceramic Capacitors MLCC - SMD/SMT 100nF 10V 0402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, lib:C0402, F.Cu at (150.5, 105.0)
- added C30: Multilayer Ceramic Capacitors MLCC - SMD/SMT 2.2uF 16V 0402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, lib:C0402, F.Cu at (140.1, 118.6)
- added C31: Multilayer Ceramic Capacitors MLCC - SMD/SMT 100nF 10V 0402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, lib:C0402, F.Cu at (133.7, 123.0)
- added C32: Multilayer Ceramic Capacitors MLCC - SMD/SMT 22nF 50V 0805 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, lib:C0805, F.Cu at (143.9, 124.6)
- added C33: Multilayer Ceramic Capacitors MLCC - SMD/SMT 100nF 50V 0603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, lib:C0603, F.Cu at (143.8, 122.5)
- added C34: Multilayer Ceramic Capacitors MLCC - SMD/SMT 1uF 6.3V 0402 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, lib:C0402, F.Cu at (178.8, 116.9)
- added C35: Multilayer Ceramic Capacitors MLCC - SMD/SMT 100nF 10V 0402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, lib:C0402, F.Cu at (112.0, 88.9)
- added C36: Multilayer Ceramic Capacitors MLCC - SMD/SMT 100nF 10V 0402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, lib:C0402, F.Cu at (113.0, 88.9)
- added C37: Multilayer Ceramic Capacitors MLCC - SMD/SMT 100nF 10V 0402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, lib:C0402, F.Cu at (107.9, 94.6)
- added C38: Multilayer Ceramic Capacitors MLCC - SMD/SMT 22nF 25V 0402 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, lib:C0402, F.Cu at (105.2, 88.9)
- added C39: Multilayer Ceramic Capacitors MLCC - SMD/SMT 22nF 25V 0402 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, lib:C0402, F.Cu at (109.0, 94.6)
- added C4: Multilayer Ceramic Capacitors MLCC - SMD/SMT 100nF 10V 0402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, lib:C0402, F.Cu at (146.0, 103.5)
- added C40: Multilayer Ceramic Capacitors MLCC - SMD/SMT 100nF 10V 0402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, lib:C0402, F.Cu at (119.0, 104.0)
- added C41: Multilayer Ceramic Capacitors MLCC - SMD/SMT 10uF 16V 1206 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, lib:C1206, F.Cu at (114.3, 100.8)
- added C42: Multilayer Ceramic Capacitors MLCC - SMD/SMT 10uF 16V 1206 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, lib:C1206, F.Cu at (105.1, 102.8)
- added C43: Multilayer Ceramic Capacitors MLCC - SMD/SMT 100nF 10V 0402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, lib:C0402, F.Cu at (103.4, 104.2)
- added C44: Multilayer Ceramic Capacitors MLCC - SMD/SMT 100nF 10V 0402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, lib:C0402, F.Cu at (109.8, 111.2)
- added C45: Multilayer Ceramic Capacitors MLCC - SMD/SMT 100nF 10V 0402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, lib:C0402, F.Cu at (118.8, 110.9)
- added C46: Multilayer Ceramic Capacitors MLCC - SMD/SMT 100nF 10V 0402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, lib:C0402, F.Cu at (109.4, 109.6)
- added C5: Multilayer Ceramic Capacitors MLCC - SMD/SMT 100nF 10V 0402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, lib:C0402, F.Cu at (107.0, 118.0)
- added C6: Multilayer Ceramic Capacitors MLCC - SMD/SMT 100nF 10V 0402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, lib:C0402, F.Cu at (106.9, 123.1)
- added C7: Multilayer Ceramic Capacitors MLCC - SMD/SMT 100nF 10V 0402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, lib:C0402, F.Cu at (109.0, 114.5)
- added C8: Multilayer Ceramic Capacitors MLCC - SMD/SMT 270pF 50V 0402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, lib:C0402, F.Cu at (106.9, 120.5)
- added C9: Multilayer Ceramic Capacitors MLCC - SMD/SMT 1uF 6.3V 0402 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, lib:C0402, F.Cu at (142.0, 105.9)
- added J1: , lib:CONN-TH_XT30PW-M, F.Cu at (158.4, 138.5)
- added L1: 1.23A 3.3uH ±20% SMD Power Inductors ROHS, lib:ato-04ea3db2-4b2f-45a6-9113-aa1f8beaa754, F.Cu at (105.9, 107.3)
- added LED1: , lib:LED0603-RD, F.Cu at (167.6, 50.0)
- added LED2: , lib:LED0603-RD, F.Cu at (138.5, 118.6)
- added Q1: , lib:SOT-23-3_L2.9-W1.3-P1.90-LS2.4-BR, F.Cu at (107.9, 103.1)
- added R1: Chip Resistor - Surface Mount 4.7KOhms ±5% 1/16W 0402 RoHS, lib:R0402, F.Cu at (106.9, 56.3)
- added R10: Chip Resistor - Surface Mount 10KOhms ±5% 1/16W 0402 RoHS, lib:R0402, F.Cu at (142.0, 91.3)
- added R11: Chip Resistor - Surface Mount 10KOhms ±5% 1/16W 0402 RoHS, lib:R0402, F.Cu at (142.0, 94.5)
- added R12: Chip Resistor - Surface Mount 10KOhms ±5% 1/16W 0402 RoHS, lib:R0402, F.Cu at (142.0, 93.5)
- added R13: Chip Resistor - Surface Mount 10KOhms ±5% 1/16W 0402 RoHS, lib:R0402, F.Cu at (154.4, 93.3)
- added R14: Chip Resistor - Surface Mount 10KOhms ±5% 1/16W 0402 RoHS, lib:R0402, F.Cu at (154.4, 94.4)
- added R15: Chip Resistor - Surface Mount 10KOhms ±5% 1/16W 0402 RoHS, lib:R0402, F.Cu at (154.4, 91.2)
- added R16: Chip Resistor - Surface Mount 10KOhms ±5% 1/16W 0402 RoHS, lib:R0402, F.Cu at (154.4, 92.3)
- added R17: Chip Resistor - Surface Mount 10KOhms ±5% 1/16W 0402 RoHS, lib:R0402, F.Cu at (154.4, 89.1)
- added R18: Chip Resistor - Surface Mount 10KOhms ±5% 1/16W 0402 RoHS, lib:R0402, F.Cu at (154.4, 90.2)
- added R19: Chip Resistor - Surface Mount 10KOhms ±5% 1/16W 0402 RoHS, lib:R0402, F.Cu at (154.4, 87.0)
- added R2: Chip Resistor - Surface Mount 4.7KOhms ±5% 1/16W 0402 RoHS, lib:R0402, F.Cu at (103.9, 56.3)
- added R20: Chip Resistor - Surface Mount 10KOhms ±5% 1/16W 0402 RoHS, lib:R0402, F.Cu at (154.4, 88.1)
- added R21: Chip Resistor - Surface Mount 51Ohms ±5% 1/16W 0402 RoHS, lib:R0402, F.Cu at (105.4, 117.3)
- added R22: Chip Resistor - Surface Mount 51Ohms ±5% 1/16W 0402 RoHS, lib:R0402, F.Cu at (105.4, 118.6)
- added R23: Chip Resistor - Surface Mount 11KOhms ±5% 1/16W 0402 RoHS, lib:R0402, F.Cu at (116.7, 57.6)
- added R24: Chip Resistor - Surface Mount 0Ohms ±5% 1/16W 0402 RoHS, lib:R0402, F.Cu at (151.0, 80.5)
- added R25: Chip Resistor - Surface Mount 0Ohms ±5% 1/16W 0402 RoHS, lib:R0402, F.Cu at (150.0, 80.5)
- added R26: Chip Resistor - Surface Mount 1KOhms ±5% 1/16W 0402 RoHS, lib:R0402, F.Cu at (177.6, 64.5)
- added R27: Chip Resistor - Surface Mount 27KOhms ±5% 1/16W 0402 RoHS, lib:R0402, F.Cu at (165.7, 60.6)
- added R28: Chip Resistor - Surface Mount 27KOhms ±5% 1/16W 0402 RoHS, lib:R0402, F.Cu at (166.8, 60.6)
- added R29: Chip Resistor - Surface Mount 11KOhms ±5% 1/16W 0402 RoHS, lib:R0402, F.Cu at (178.7, 60.0)
- added R3: Chip Resistor - Surface Mount 4.7KOhms ±5% 1/16W 0402 RoHS, lib:R0402, F.Cu at (152.2, 56.3)
- added R30: Chip Resistor - Surface Mount 10KOhms ±5% 1/16W 0402 RoHS, lib:R0402, F.Cu at (166.8, 67.6)
- added R31: Chip Resistor - Surface Mount 0Ohms ±5% 1/16W 0402 RoHS, lib:R0402, F.Cu at (153.2, 80.5)
- added R32: Chip Resistor - Surface Mount 0Ohms ±5% 1/16W 0402 RoHS, lib:R0402, F.Cu at (154.2, 80.5)
- added R33: Chip Resistor - Surface Mount 18KOhms ±5% 1/16W 0402 RoHS, lib:R0402, F.Cu at (161.3, 49.8)
- added R34: Chip Resistor - Surface Mount 10KOhms ±5% 1/16W 0402 RoHS, lib:R0402, F.Cu at (163.3, 49.8)
- added R35: Chip Resistor - Surface Mount 120Ohms ±5% 1/16W 0402 RoHS, lib:R0402, F.Cu at (167.6, 52.9)
- added R36: Chip Resistor - Surface Mount 110KOhms ±5% 1/16W 0402 RoHS, lib:R0402, F.Cu at (144.3, 126.0)
- added R37: Chip Resistor - Surface Mount 1.1KOhms ±5% 1/16W 0402 RoHS, lib:R0402, F.Cu at (135.4, 118.1)
- added R38: Chip Resistor - Surface Mount 120Ohms ±5% 1/16W 0402 RoHS, lib:R0402, F.Cu at (137.1, 118.1)
- added R39: Chip Resistor - Surface Mount 0.12Ohms ±5% 1/8W 0805 RoHS, lib:R0805, F.Cu at (137.2, 130.6)
- added R4: Chip Resistor - Surface Mount 4.7KOhms ±5% 1/16W 0402 RoHS, lib:R0402, F.Cu at (149.3, 56.3)
- added R40: Chip Resistor - Surface Mount 0.12Ohms ±5% 1/8W 0805 RoHS, lib:R0805, F.Cu at (140.0, 130.6)
- added R41: Chip Resistor - Surface Mount 110KOhms ±5% 1/16W 0402 RoHS, lib:R0402, F.Cu at (133.7, 125.4)
- added R42: Chip Resistor - Surface Mount 1KOhms ±5% 1/16W 0402 RoHS, lib:R0402, F.Cu at (129.4, 128.1)
- added R43: Chip Resistor - Surface Mount 1KOhms ±5% 1/16W 0402 RoHS, lib:R0402, F.Cu at (129.3, 125.6)
- added R44: Chip Resistor - Surface Mount 1KOhms ±5% 1/16W 0402 RoHS, lib:R0402, F.Cu at (129.4, 123.0)
- added R45: Chip Resistor - Surface Mount 1KOhms ±5% 1/16W 0402 RoHS, lib:R0402, F.Cu at (129.3, 120.5)
- added R46: Chip Resistor - Surface Mount 1KOhms ±5% 1/16W 0402 RoHS, lib:R0402, F.Cu at (169.7, 88.9)
- added R47: Chip Resistor - Surface Mount 1KOhms ±5% 1/16W 0402 RoHS, lib:R0402, F.Cu at (169.7, 86.4)
- added R48: Chip Resistor - Surface Mount 1KOhms ±5% 1/16W 0402 RoHS, lib:R0402, F.Cu at (169.7, 83.8)
- added R49: Chip Resistor - Surface Mount 1KOhms ±5% 1/16W 0402 RoHS, lib:R0402, F.Cu at (169.7, 81.3)
- added R5: Chip Resistor - Surface Mount 10KOhms ±5% 1/16W 0402 RoHS, lib:R0402, F.Cu at (142.0, 88.1)
- added R50: Chip Resistor - Surface Mount 1KOhms ±5% 1/16W 0402 RoHS, lib:R0402, F.Cu at (169.5, 112.6)
- added R51: Chip Resistor - Surface Mount 1KOhms ±5% 1/16W 0402 RoHS, lib:R0402, F.Cu at (169.5, 110.1)
- added R52: Chip Resistor - Surface Mount 1KOhms ±5% 1/16W 0402 RoHS, lib:R0402, F.Cu at (169.5, 107.5)
- added R53: Chip Resistor - Surface Mount 1KOhms ±5% 1/16W 0402 RoHS, lib:R0402, F.Cu at (169.5, 105.0)
- added R54: Chip Resistor - Surface Mount 1KOhms ±5% 1/16W 0402 RoHS, lib:R0402, F.Cu at (130.9, 79.5)
- added R55: Chip Resistor - Surface Mount 1KOhms ±5% 1/16W 0402 RoHS, lib:R0402, F.Cu at (128.3, 79.5)
- added R56: Chip Resistor - Surface Mount 1KOhms ±5% 1/16W 0402 RoHS, lib:R0402, F.Cu at (125.7, 79.5)
- added R57: Chip Resistor - Surface Mount 1KOhms ±5% 1/16W 0402 RoHS, lib:R0402, F.Cu at (123.2, 79.5)
- added R58: Chip Resistor - Surface Mount 20KOhms ±5% 1/16W 0402 RoHS, lib:R0402, F.Cu at (109.5, 105.9)
- added R59: Chip Resistor - Surface Mount 8.2KOhms ±5% 1/16W 0402 RoHS, lib:R0402, F.Cu at (109.5, 107.9)
- added R6: Chip Resistor - Surface Mount 10KOhms ±5% 1/16W 0402 RoHS, lib:R0402, F.Cu at (142.0, 87.0)
- added R60: Chip Resistor - Surface Mount 100Ohms ±5% 1/16W 0402 RoHS, lib:R0402, F.Cu at (108.3, 111.7)
- added R61: Chip Resistor - Surface Mount 100Ohms ±5% 1/16W 0402 RoHS, lib:R0402, F.Cu at (108.3, 110.6)
- added R62: Chip Resistor - Surface Mount 100Ohms ±5% 1/16W 0402 RoHS, lib:R0402, F.Cu at (120.4, 110.4)
- added R63: Chip Resistor - Surface Mount 100Ohms ±5% 1/16W 0402 RoHS, lib:R0402, F.Cu at (120.4, 111.5)
- added R7: Chip Resistor - Surface Mount 10KOhms ±5% 1/16W 0402 RoHS, lib:R0402, F.Cu at (142.0, 90.2)
- added R8: Chip Resistor - Surface Mount 10KOhms ±5% 1/16W 0402 RoHS, lib:R0402, F.Cu at (142.0, 89.2)
- added R9: Chip Resistor - Surface Mount 10KOhms ±5% 1/16W 0402 RoHS, lib:R0402, F.Cu at (142.0, 92.4)
- added U1: , lib:USB-C-SMD_KH-TYPE-C-16P, F.Cu at (105.6, 51.9)
- added U10: , lib:KEY-SMD_4P-L4.2-W3.2-P2.20-LS4.6, F.Cu at (114.5, 59.6)
- added U11: , lib:HDR-SMD_10P-P1.27-V-M-R2-C5-LS5.3, F.Cu at (143.0, 63.0)
- added U12: , lib:LQFN-56_L7.0-W7.0-P0.4-EP, F.Cu at (171.6, 64.3)
- added U13: , lib:OSC-SMD_4P-L3.2-W2.5-BL, F.Cu at (179.9, 65.7)
- added U14: , lib:SOIC-8_L5.3-W5.3-P1.27-LS8.0-BL, F.Cu at (162.7, 64.3)
- added U15: , lib:KEY-SMD_4P-L4.2-W3.2-P2.20-LS4.6, F.Cu at (180.2, 57.3)
- added U16: , lib:KEY-SMD_4P-L4.2-W3.2-P2.20-LS4.6, F.Cu at (158.3, 69.1)
- added U17: , lib:SOT-23-5_L3.0-W1.7-P0.95-LS2.8-BL, F.Cu at (162.2, 52.4)
- added U18: , lib:QFN-28_L5.0-W5.0-P0.50-BL-EP, F.Cu at (138.5, 124.5)
- added U19: , lib:HDR-SMD_8P-P2.54-V-M-R2-C4-LS7.4, F.Cu at (123.8, 124.3)
- added U2: , lib:USB-C-SMD_KH-TYPE-C-16P, F.Cu at (151.0, 51.9)
- added U20: , lib:CONN-TH_4P-P5.08_DIBO_DB128V-5.08, F.Cu at (137.2, 141.0)
- added U21: , lib:TF-SMD_TF-01A, F.Cu at (181.9, 81.7)
- added U22: , lib:HDR-SMD_8P-P2.54-V-M-R2-C4-LS7.4, F.Cu at (164.1, 85.1)
- added U23: , lib:GPSM-SMD_ATGM336H-TR, F.Cu at (177.8, 109.2)
- added U24: , lib:IPEX-SMD_BWIPX-1-001E, F.Cu at (174.4, 116.9)
- added U25: , lib:HDR-SMD_8P-P2.54-V-M-R2-C4-LS7.4, F.Cu at (163.9, 108.8)
- added U26: , lib:TSSOP-14_L5.0-W4.4-P0.65-LS6.4-BL, F.Cu at (108.6, 89.0)
- added U27: , lib:CONN-TH_DB125-2.54-2P-GN, F.Cu at (94.7, 90.2)
- added U28: , lib:HDR-SMD_8P-P2.54-V-M-R2-C4-LS7.4, F.Cu at (127.0, 85.1)
- added U29: , lib:SOP-16_L10.0-W3.9-P1.27-LS6.0-BL, F.Cu at (114.3, 107.1)
- added U3: , lib:TSSOP-24_L7.8-W4.4-P0.65-LS6.4-BL, F.Cu at (148.1, 90.4)
- added U30: , lib:CONN-TH_XY308-2.54-4P, F.Cu at (94.8, 106.0)
- added U4: , lib:LGA-8_BME280_BL, F.Cu at (152.5, 105.0)
- added U5: , lib:LGA-12_L2.0-W2.0-P0.50-BL, F.Cu at (146.1, 105.4)
- added U6: , lib:SOP-16_L9.9-W3.9-P1.27-LS6.0-BL, F.Cu at (111.7, 120.6)
- added U7: , lib:CONN-TH_XY308-2.54-4P, F.Cu at (95.0, 121.2)
- added U8: , lib:DFN-6_L2.4-W2.4-P0.80-TL-EP, F.Cu at (139.8, 105.4)
- added U9: , lib:WIRELM-SMD_ESP32-S3-WROOM-1, F.Cu at (127.7, 63.2)
Routing:
- net vcc: track 0.00 -> 182.8 mm, vias 0 -> 27
- net vcc-1: track 0.00 -> 143.8 mm, vias 0 -> 3
- net gnd: track 0.00 -> 130.9 mm, vias 0 -> 65
- net clock: track 0.00 -> 89.3 mm, vias 0 -> 2
- net data: track 0.00 -> 87.3 mm, vias 0 -> 2
- net dir: track 0.00 -> 87.2 mm, vias 0 -> 2
- net step: track 0.00 -> 84.3 mm, vias 0 -> 2
- net tx: track 0.00 -> 65.9 mm
- net rx: track 0.00 -> 65.4 mm, vias 0 -> 2
- net scl-3: track 0.00 -> 60.8 mm
- net sda-3: track 0.00 -> 57.0 mm
- net scl: track 0.00 -> 49.8 mm, vias 0 -> 2
- net scl-9: track 0.00 -> 49.1 mm, vias 0 -> 2
- net sda-9: track 0.00 -> 48.0 mm, vias 0 -> 2
- net sda: track 0.00 -> 47.6 mm, vias 0 -> 2
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- added copper zone on F.Cu, net gnd
- added copper zone on In2.Cu, net gnd
- added copper zone on In1.Cu, net vcc
Other:
- board size 225.7 x 100.8 mm -> 100 x 100 mm
- copper layers 2 -> 4
- board text added: "3V3"
- board text added: "3v3"
- board text added: "A1"
- board text added: "A2"
- board text added: "ATGM336"
- board text added: "B1"
- board text added: "B2"
- board text added: "BME280"
- board text added: "BOOT"
- board text added: "CS"
- board text added: "DIR"
- board text added: "ESP32"
- board text added: "FORCE+"
- board text added: "FORCE-"
- board text added: "GND"
- board text added: "LIS2DH"
- board text added: "MAX31856"
- board text added: "MISO"
- board text added: "MOSI"
- board text added: "RP2040"
- board text added: "RUN"
- board text added: "RX"
- board text added: "SCK"
- board text added: "SCL"
- board text added: "SDA"
- board text added: "SENSE+"
- board text added: "SENSE-"
- board text added: "SGP40"
- board text added: "STEP"
- board text added: "TMC2209"
- board text added: "TX"
- board text added: "VBUS"
- board text added: "VCC"
