File: elec/layout/default/the-everything-sensor.kicad_pcb (KiCad board)
At the start: 4 copper layers, 100 x 100 mm, 144 parts

Commit message: cleanup silkscreen
Routing:
- net gnd: vias 65 -> 64
Other:
- board text added: "The Everything Sensor"
